File: project/candidate.kicad_pcb (KiCad board)
At the start: 4 copper layers, 105.6 x 69 mm, 164 parts, among them J4 Conn_01x04_Pin, J5 Conn_01x04_Pin, Q15 Q_Dual_NPN_PNP_B1E2B2C2E1C1, Q16 Q_Dual_NPN_PNP_B1E2B2C2E1C1, Q17 Q_Dual_NPN_PNP_B1E2B2C2E1C1, Q18 Q_Dual_NPN_PNP_B1E2B2C2E1C1, Q19 Q_Dual_NPN_PNP_B1E2B2C2E1C1, Q20 Q_Dual_NPN_PNP_B1E2B2C2E1C1, Q21 Q_Dual_NPN_PNP_B1E2B2C2E1C1, Q22 Q_Dual_NPN_PNP_B1E2B2C2E1C1, Q23 Q_Dual_NPN_PNP_B1E2B2C2E1C1, Q24 Q_Dual_NPN_PNP_B1E2B2C2E1C1, Q25 Q_Dual_NPN_PNP_B1E2B2C2E1C1, Q26 Q_Dual_NPN_PNP_B1E2B2C2E1C1, Q27 Q_Dual_NPN_PNP_B1E2B2C2E1C1, Q28 Q_Dual_NPN_PNP_B1E2B2C2E1C1, Q29 Q_Dual_NPN_PNP_B1E2B2C2E1C1, SW1 SW_Push, SW2 SW_Push, SW3 SW_Push, U1 74AUP1G80, U10 NMUX1308BQ, U11 NMUX1308BQ, U12 NMUX1308BQ, U13 NMUX1308BQ, U14 NMUX1308BQ, U15 NMUX1308BQ, U16 NMUX1308BQ, U17 74AUP1G80, U18 74AHC1G86, U19 74AUP1G80, U20 74AUP1G80, U21 74LV1T08GV, U22 CD74HC283M96, U23 74LV1T08GV, U24 74LVC1GU04DRL, U25 ESP32-S3-MINI-1, U26 74LVC1GU04DRL, U27 74LV1T08GV, U28 CD74HC283M96, U29 NMUX1308BQ, U3 74AHC1G86, U30 NMUX1308BQ, U31 NMUX1308BQ, U32 NMUX1308BQ, U33 74AUP1G80, U34 74AUP1G80, U35 NMUX1308BQ, U36 NMUX1308BQ, U37 74AUP1G80, U38 74AUP1G80, U39 NMUX1308BQ, U4 74AUP1G80, U40 NMUX1308BQ, U41 NMUX1308BQ, U42 NMUX1308BQ, U43 NMUX1308BQ, U44 NMUX1308BQ, U45 74AUP1G80, U46 74AUP1G80, U47 74AUP1G80, U48 74AUP1G80, U49 74AUP1G80, U5 74AUP1G80, U50 74AUP1G80, U51 74LV1T08GV, U52 74AHC1G86, U53 74LVC1GU04DRL, U54 74LVC1GU04DRL, U55 74AHC1G86, U56 74AHC1G86, U57 74LVC1GU04DRL, U58 74LVC1GU04DRL, U59 74LV1T08GV, U6 74AUP1G80, U60 74AHC1G86, U61 74LVC1GU04DRL, U62 74LV1T08GV, U63 74LV1T08GV, U64 NMUX1308BQ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

Commit message: Update measured candidate to 52 unconnected items; retain unresolved findings
Routing:
- net wir1: track 0.00 -> 35.9 mm, vias 0 -> 2
- net GND: track 239.8 -> 261.3 mm, vias 120 -> 121
- net R_en: track 87.0 -> 108.4 mm, vias 3 -> 6
- net IO6: track 312.4 -> 295.5 mm
- net out_4: track 24.0 -> 31.8 mm, vias 2 -> 5
- net Net-(U28-CIN): track 0.00 -> 4.99 mm
- net Net-(Q25A-E1): track 44.1 -> 44.9 mm
- net +3.3V: vias 10 -> 12

Commit message: Freeze measured candidate: 48 unconnected items, unresolved validity
Routing:
- net Net-(Q24A-E1): track 0.00 -> 29.7 mm
- net out_1: track 0.00 -> 23.7 mm, vias 0 -> 2
- net ???: track 0.00 -> 22.9 mm, vias 0 -> 2
- net IO8: track 262.1 -> 284.6 mm, vias 13 -> 14
- net Net-(U25-IO16): track 0.00 -> 11.6 mm
- net en: track 0.00 -> 7.29 mm, vias 0 -> 1
- net R_en: track 108.4 -> 109.0 mm

Commit message: Freeze measured candidate: 47 unconnected items, unresolved validity
Routing:
- net GND: track 261.3 -> 265.6 mm, vias 121 -> 122
Changed lines of the file:
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@@
-	)
-	(segment
-		(start 60.75 22.75)
-		(end 65.75 34.75)
-		(width 0.15)
-		(layer "F.Cu")
-		(net "GND")
 	)
 	(segment
@@
 	)
 	(segment
-		(start 65.75 35.75)
-		(end 64.25 37)
-		(width 0.15)
-		(layer "F.Cu")
-		(net "GND")
-	)
-	(segment
 		(start 74.5 40.6625)
 		(end 74.5 39.7625)
@@
 	)
 	(segment
-		(start 65.75 34.75)
-		(end 65.75 35.75)
-		(width 0.15)
-		(layer "F.Cu")
-		(net "GND")
-	)
-	(segment
 		(start 34.4 17.3375)
 		(end 36 17.3375)
@@
 		(end 20.975 16.5)
 		(width 0.17)
-		(layer "F.Cu")
-		(net "GND")
-	)
-	(segment
-		(start 60.025 22.175)
-		(end 60.75 22.75)
-		(width 0.15)
 		(layer "F.Cu")
 		(net "GND")
@@
 	)
 	(segment
+		(start 60.025 22.175)
+		(end 43.75 22.175)
+		(width 0.15)
+		(layer "F.Cu")
+		(net "GND")
+	)
+	(segment
 		(start 7.5 19.049999)
 		(end 6.5 18.775)
@@
 	)
 	(via
+		(at 43.75 22.175)
+		(size 0.6)
+		(drill 0.3)
+		(layers "F.Cu" "B.Cu")
+		(net "GND")
+	)
+	(via
 		(at 41.075 47.5)
 		(size 0.6)
@@
 		(net "GND")
 	)
+	(segment
+		(start 43.75 22.175)
+		(end 44.5 24.25)
+		(width 0.17)
+		(layer "In1.Cu")
+		(net "GND")
+	)
+	(segment
+		(start 44.5 24.25)
+		(end 43.4 26.775)
+		(width 0.17)
+		(layer "In1.Cu")
+		(net "GND")
+	)
